File: MCMP_Projeto_Final.brd (EAGLE design)
At the start: 144.8 x 111.4 mm, 66 parts, among them IC1 PIC16F877A-I_P, IC2 LM7805ACT, IC3 L293D, IC4 L293D, J1 694106301002, K1 SRD-05VDC-SL-C, K2 SRD-05VDC-SL-C, K3 SRD-05VDC-SL-C, K5 SRD-05VDC-SL-C, Q1 2N1711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

Commit message: 1.0.0.060520210411
Parts:
- added J3: (no value), Wurth_Connectors_WR-PHD:62000211121
- added R2: 330, Resistor_Capacitor:RES_0805
Connections:
- new net N$10: IC1.33, J3.1, R2.1
- net GND: now also R2.2
- net VCC5: now also J3.2
Routing:
- net GND: track 754.8 -> 766.1 mm, vias 0 -> 1
- net N$10: track 0.00 -> 9.19 mm
Changed lines of the file:
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@@
 <drawing>
 <settings>
-<setting alwaysvectorfont="yes"/>
+<setting alwaysvectorfont="no"/>
 <setting verticaltext="up"/>
 </settings>
@@
 <element name="U$5" library="adafruit" library_urn="urn:adsk.eagle:library:420" package="FIDUCIAL_1MM" package3d_urn="urn:adsk.eagle:package:6240632/1" value="FIDUCIAL" x="21.59" y="-8.89" smashed="yes"/>
 <element name="U$6" library="adafruit" library_urn="urn:adsk.eagle:library:420" package="FIDUCIAL_1MM" package3d_urn="urn:adsk.eagle:package:6240632/1" value="FIDUCIAL" x="24.13" y="-8.89" smashed="yes" rot="MR0"/>
+<element name="J3" library="Wurth_Connectors_WR-PHD" library_urn="urn:adsk.eagle:library:14804658" package="62000211121" package3d_urn="urn:adsk.eagle:package:14805726/2" value="" x="106.68" y="55.88" smashed="yes" rot="R270">
+<attribute name="DATASHEET-URL" value="https://katalog.we-online.com/em/datasheet/62000211121.pdf" x="106.68" y="55.88" size="1.778" layer="27" rot="R270" display="off"/>
+<attribute name="GENDER" value="Pin Header" x="106.68" y="55.88" size="1.778" layer="27" rot="R270" display="off"/>
+<attribute name="IR" value="2A" x="106.68" y="55.88" size="1.778" layer="27" rot="R270" display="off"/>
+<attribute name="MATES" value="WR-PHD 2.0mm Socket Header" x="106.68" y="55.88" size="1.778" layer="27" rot="R270" display="off"/>
+<attribute name="NAME" x="106.7449" y="58.7164" size="0.8128" layer="25" rot="R270" align="bottom-right"/>
+<attribute name="PACKAGING" value="Bag" x="106.68" y="55.88" size="1.778" layer="27" rot="R270" display="off"/>
+<attribute name="PART-NUMBER" value=" 62000211121 " x="106.68" y="55.88" size="1.778" layer="27" rot="R270" display="off"/>
+<attribute name="PINS" value=" 2 " x="106.68" y="55.88" size="1.778" layer="27" rot="R270" display="off"/>
+<attribute name="ROWS" value="Single" x="106.68" y="55.88" size="1.778" layer="27" rot="R270" display="off"/>
+<attribute name="TYPE" value="Straight" x="106.68" y="55.88" size="1.778" layer="27" rot="R270" display="off"/>
+<attribute name="VALUE" x="105.387" y="58.7164" size="0.8128" layer="27" rot="R270" align="bottom-right"/>
+</element>
+<element name="R2" library="Resistor_Capacitor" library_urn="urn:adsk.eagle:library:15122775" package="RES_0805" package3d_urn="urn:adsk.eagle:package:10872899/3" value="330" x="111.76" y="55.88" smashed="yes" rot="R270">
+<attribute name="CREATED_BY" value="PCBLayout.com" x="111.76" y="55.88" size="1.778" layer="27" rot="R270" display="off"/>
+<attribute name="DIGIKEY_PART_NUMBER" value="541-0.0ATR-ND" x="111.76" y="55.88" size="1.778" layer="27" rot="R270" display="off"/>
+<attribute name="MANUFACTURER" value="Vishay Dale" x="111.76" y="55.88" size="1.778" layer="27" rot="R270" display="off"/>
+<attribute name="MPN" value="CRCW08050000Z0EA" x="111.76" y="55.88" size="1.778" layer="27" rot="R270" display="off"/>
+<attribute name="NAME" x="113.03" y="58.166" size="0.87" layer="25" ratio="10" rot="R270"/>
+<attribute name="PACKAGE" value="SMD 0805" x="111.76" y="55.88" size="1.778" layer="27" rot="R270" display="off"/>
+<attribute name="VALUE" x="109.728" y="58.166" size="0.87" layer="27" ratio="10" rot="R270"/>
+</element>
 </elements>
 <signals>
@@
 <wire x1="134.62" y1="43.18" x2="128.27" y2="43.18" width="0.6096" layer="16"/>
 <wire x1="53.34" y1="82.55" x2="53.34" y2="91.44" width="1.27" layer="16"/>
+<wire x1="102.998" y1="50.8" x2="106.68" y2="50.8" width="0.6096" layer="16"/>
+<contactref element="R2" pad="2"/>
+<wire x1="106.68" y1="50.8" x2="109.22" y2="53.34" width="0.6096" layer="16"/>
+<wire x1="109.22" y1="53.34" x2="109.22" y2="54.61" width="0.6096" layer="16"/>
+<via x="109.22" y="54.61" extent="1-16" drill="0.35"/>
+<wire x1="111.76" y1="54.905" x2="111.465" y2="54.61" width="0.6096" layer="1"/>
+<wire x1="111.465" y1="54.61" x2="109.22" y2="54.61" width="0.6096" layer="1"/>
 <wire x1="8.89" y1="81.28" x2="9.07" y2="81.46" width="0" layer="19" extent="1-1"/>
 </signal>
@@
 <wire x1="122.0622" y1="46.4178" x2="122.0622" y2="46.4517625" width="0.6096" layer="1"/>
 <wire x1="122.0622" y1="46.4517625" x2="115.6039625" y2="52.91" width="0.6096" layer="1"/>
-<wire x1="115.6039625" y1="52.91" x2="106.68" y2="52.91" width="0.6096" layer="1"/>
+<wire x1="115.6039625" y1="52.91" x2="109.22" y2="52.91" width="0.6096" layer="1"/>
+<wire x1="109.22" y1="52.91" x2="106.68" y2="52.91" width="0.6096" layer="1"/>
 <wire x1="123.29814375" y1="76.2" x2="123.19" y2="76.63" width="0.6096" layer="1"/>
 <wire x1="87.502" y1="48.26" x2="87.072" y2="47.83" width="0.6096" layer="1"/>
@@
 <wire x1="128.27" y1="40.64" x2="135.89" y2="33.02" width="0.6096" layer="1"/>
 <wire x1="135.89" y1="33.02" x2="135.89" y2="27.94" width="0.6096" layer="1"/>
+<contactref element="J3" pad="2"/>
+<wire x1="106.68" y1="52.91" x2="106.68" y2="54.88" width="0" layer="19" extent="1-1"/>
 </signal>
 <signal name="N$2">
@@
 <wire x1="142.24" y1="19.05" x2="142.24" y2="76.2" width="0.6096" layer="16"/>
 </signal>
+<signal name="N$10">
+<contactref element="IC1" pad="33"/>
+<contactref element="J3" pad="1"/>
+<contactref element="R2" pad="1"/>
+<wire x1="102.998" y1="55.88" x2="103.998" y2="56.88" width="0.6096" layer="1"/>
+<wire x1="103.998" y1="56.88" x2="106.68" y2="56.88" width="0.6096" layer="1"/>
+<wire x1="111.76" y1="56.855" x2="111.735" y2="56.88" width="0.6096" layer="1"/>
+<wire x1="111.735" y1="56.88" x2="106.68" y2="56.88" width="0.6096" layer="1"/>
+</signal>
 </signals>
