File: MCMP_Projeto_Final.sch (EAGLE design)
At the start: 62 parts, among them IC1 PIC16F877A-I_P, IC2 LM7805ACT, IC3 L293D, IC4 L293D, J1 694106301002, K1 SRD-05VDC-SL-C, K2 SRD-05VDC-SL-C, K3 SRD-05VDC-SL-C, K5 SRD-05VDC-SL-C, Q1 2N1711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

Commit message: 1.0.0.060520210411
Parts:
- added J3: (no value), Wurth_Connectors_WR-PHD:6200XX11121_62000211121
- added R2: 330, Resistor_Capacitor:CRCW08050000Z0EA
Connections:
- new net N$10: IC1.RB0/INT, J3.1, R2.1
- net GND: now also R2.2
- net VCC5: now also J3.2
Changed lines of the file:
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@@
 <setting verticaltext="up"/>
 </settings>
-<grid distance="0.1" unitdist="inch" unit="inch" style="lines" multiple="1" display="no" altdistance="0.01" altunitdist="inch" altunit="inch"/>
+<grid distance="0.1" unitdist="mm" unit="mm" style="lines" multiple="1" display="no" altdistance="0.1" altunitdist="mm" altunit="mm"/>
 <layers>
 <layer number="1" name="Top" color="4" fill="1" visible="no" active="no"/>
@@
 <part name="U$5" library="adafruit" library_urn="urn:adsk.eagle:library:420" deviceset="FIDUCIAL" device="" package3d_urn="urn:adsk.eagle:package:6240632/1"/>
 <part name="U$6" library="adafruit" library_urn="urn:adsk.eagle:library:420" deviceset="FIDUCIAL" device="" package3d_urn="urn:adsk.eagle:package:6240632/1"/>
+<part name="J3" library="Wurth_Connectors_WR-PHD" library_urn="urn:adsk.eagle:library:14804658" deviceset="6200XX11121_62000211121" device="" package3d_urn="urn:adsk.eagle:package:14805726/2"/>
+<part name="R2" library="Resistor_Capacitor" library_urn="urn:adsk.eagle:library:15122775" deviceset="CRCW08050000Z0EA" device="" package3d_urn="urn:adsk.eagle:package:10872899/3" value="330"/>
 </parts>
 <sheets>
@@
 <instance part="U$5" gate="G$1" x="-55.88" y="-43.18" smashed="yes"/>
 <instance part="U$6" gate="G$1" x="-63.5" y="-43.18" smashed="yes"/>
+<instance part="J3" gate="G$1" x="142.24" y="108.712" smashed="yes" rot="R270">
+<attribute name="NAME" x="141.035" y="113.702" size="1.016" layer="95" rot="R270" align="bottom-right"/>
+<attribute name="VALUE" x="139.23" y="113.662" size="1.016" layer="96" rot="R270" align="bottom-right"/>
+</instance>
+<instance part="R2" gate="G$1" x="149.52" y="116.44" smashed="yes">
+<attribute name="NAME" x="145.71" y="117.9386" size="1.778" layer="95"/>
+<attribute name="VALUE" x="145.71" y="113.138" size="1.778" layer="96"/>
+</instance>
 </instances>
 <busses>
@@
 <wire x1="199.3" y1="99.2" x2="172.2" y2="99.2" width="0.1524" layer="91"/>
 <wire x1="180.32" y1="129.1" x2="172.2" y2="129.1" width="0.1524" layer="91"/>
-<wire x1="172.2" y1="129.1" x2="172.2" y2="104.4" width="0.1524" layer="91"/>
+<wire x1="172.2" y1="129.1" x2="172.2" y2="116.44" width="0.1524" layer="91"/>
 <junction x="172.2" y="99.2"/>
+<wire x1="172.2" y1="116.44" x2="172.2" y2="104.4" width="0.1524" layer="91"/>
 <wire x1="172.2" y1="104.4" x2="172.2" y2="99.2" width="0.1524" layer="91"/>
 <pinref part="LED8" gate="G$1" pin="C"/>
@@
 <wire x1="137" y1="155.42" x2="137" y2="138" width="0.1524" layer="91"/>
 <junction x="137" y="138"/>
+<pinref part="R2" gate="G$1" pin="2"/>
+<wire x1="154.6" y1="116.44" x2="172.2" y2="116.44" width="0.1524" layer="91"/>
 </segment>
 </net>
@@
 <wire x1="154.9" y1="148.2" x2="154.7" y2="148.2" width="0.1524" layer="91"/>
 <pinref part="C18" gate="G$1" pin="1"/>
-<wire x1="154.7" y1="148.2" x2="124.3" y2="148.2" width="0.1524" layer="91"/>
+<wire x1="154.7" y1="148.2" x2="154.6" y2="148.2" width="0.1524" layer="91"/>
+<wire x1="154.6" y1="148.2" x2="124.3" y2="148.2" width="0.1524" layer="91"/>
 <wire x1="154.7" y1="147.14" x2="154.7" y2="148.2" width="0.1524" layer="91"/>
 <junction x="154.7" y="148.2"/>
@@
 <wire x1="154.78" y1="149.82" x2="154.78" y2="155.42" width="0.1524" layer="91"/>
 <junction x="154.78" y="149.82"/>
+<pinref part="J3" gate="G$1" pin="2"/>
+<wire x1="137.16" y1="108.712" x2="137.16" y2="106.2" width="0.1524" layer="91"/>
+<wire x1="137.16" y1="106.2" x2="162.9" y2="106.2" width="0.1524" layer="91"/>
+<wire x1="162.9" y1="106.2" x2="162.9" y2="148.2" width="0.1524" layer="91"/>
+<wire x1="162.9" y1="148.2" x2="154.7" y2="148.2" width="0.1524" layer="91"/>
 </segment>
 </net>
@@
 </segment>
 </net>
+<net name="N$10" class="0">
+<segment>
+<pinref part="IC1" gate="G$1" pin="RB0/INT"/>
+<pinref part="J3" gate="G$1" pin="1"/>
+<wire x1="113.88" y1="111.22" x2="137.16" y2="111.22" width="0.1524" layer="91"/>
+<wire x1="137.16" y1="111.22" x2="137.16" y2="111.252" width="0.1524" layer="91"/>
+<pinref part="R2" gate="G$1" pin="1"/>
+<wire x1="144.44" y1="116.44" x2="137.16" y2="116.44" width="0.1524" layer="91"/>
+<wire x1="137.16" y1="116.44" x2="137.16" y2="111.252" width="0.1524" layer="91"/>
+<junction x="137.16" y="111.252"/>
+</segment>
+</net>
